File: Compact23256.kicad_sch (KiCad schematic)
At the start: 14 parts, among them CN1 2364, U1 28C256

Commit message: Work in progress.
Parts:
- J1: footprint (none) -> Connector_PinHeader_2.54mm:PinHeader_1x03_P2.54mm_Horizontal
- JP1: value (none) -> A13; footprint (none) -> Library:SolderJumper-2_slim
- JP2: value (none) -> A14; footprint (none) -> Library:SolderJumper-2_slim
- JP3: value (none) -> CS; footprint (none) -> Library:SolderJumper-2_slim
- JP4: value (none) -> WE; footprint (none) -> Library:SolderJumper-2_slim
- SW1: value (none) -> DIP Switch; footprint (none) -> Button_Switch_SMD:SW_DIP_SPSTx04_Slide_KingTek_DSHP04TS_W7.62mm_P1.27mm
- TP3: value (none) -> CS
- TP4: value (none) -> WE; footprint (none) -> TestPoint:TestPoint_Pad_D1.5mm
Changed lines of the file:
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@@
       (effects (font (size 1.27 1.27)) (justify right))
     )
-    (property "Value" "" (id 1) (at 102.87 141.605 0)
-      (effects (font (size 1.27 1.27)) (justify right))
-    )
-    (property "Footprint" "" (id 2) (at 100.33 141.605 0)
+    (property "Value" "WE" (id 1) (at 102.87 141.605 0)
+      (effects (font (size 1.27 1.27)) (justify right))
+    )
+    (property "Footprint" "Library:SolderJumper-2_slim" (id 2) (at 100.33 141.605 0)
       (effects (font (size 1.27 1.27)) hide)
     )
@@
     (in_bom yes) (on_board yes)
     (property "Reference" "TP4" (id 0) (at 88.265 123.825 90))
-    (property "Value" "" (id 1) (at 92.71 123.825 90))
-    (property "Footprint" "" (id 2) (at 99.06 118.745 0)
+    (property "Value" "WE" (id 1) (at 92.71 123.825 90))
+    (property "Footprint" "TestPoint:TestPoint_Pad_D1.5mm" (id 2) (at 99.06 118.745 0)
       (effects (font (size 1.27 1.27)) hide)
     )
@@
       (effects (font (size 1.27 1.27)) (justify right))
     )
-    (property "Value" "" (id 1) (at 107.95 141.605 0)
-      (effects (font (size 1.27 1.27)) (justify right))
-    )
-    (property "Footprint" "" (id 2) (at 105.41 141.605 0)
+    (property "Value" "CS" (id 1) (at 107.95 141.605 0)
+      (effects (font (size 1.27 1.27)) (justify right))
+    )
+    (property "Footprint" "Library:SolderJumper-2_slim" (id 2) (at 105.41 141.605 0)
       (effects (font (size 1.27 1.27)) hide)
     )
@@
       (effects (font (size 1.27 1.27)) (justify right))
     )
-    (property "Value" "" (id 1) (at 118.11 141.605 0)
-      (effects (font (size 1.27 1.27)) (justify right))
-    )
-    (property "Footprint" "" (id 2) (at 115.57 141.605 0)
+    (property "Value" "A13" (id 1) (at 118.11 141.605 0)
+      (effects (font (size 1.27 1.27)) (justify right))
+    )
+    (property "Footprint" "Library:SolderJumper-2_slim" (id 2) (at 115.57 141.605 0)
       (effects (font (size 1.27 1.27)) hide)
     )
@@
       (effects (font (size 1.27 1.27)) (justify left))
     )
-    (property "Value" "" (id 1) (at 142.24 144.145 90)
-      (effects (font (size 1.27 1.27)) (justify left))
-    )
-    (property "Footprint" "" (id 2) (at 133.985 141.605 0)
+    (property "Value" "DIP Switch" (id 1) (at 142.24 144.145 90)
+      (effects (font (size 1.27 1.27)) (justify left))
+    )
+    (property "Footprint" "Button_Switch_SMD:SW_DIP_SPSTx04_Slide_KingTek_DSHP04TS_W7.62mm_P1.27mm" (id 2) (at 133.985 141.605 0)
       (effects (font (size 1.27 1.27)) hide)
     )
@@
       (effects (font (size 1.27 1.27)) (justify right))
     )
-    (property "Value" "" (id 1) (at 113.03 141.605 0)
-      (effects (font (size 1.27 1.27)) (justify right))
-    )
-    (property "Footprint" "" (id 2) (at 110.49 141.605 0)
+    (property "Value" "A14" (id 1) (at 113.03 141.605 0)
+      (effects (font (size 1.27 1.27)) (justify right))
+    )
+    (property "Footprint" "Library:SolderJumper-2_slim" (id 2) (at 110.49 141.605 0)
       (effects (font (size 1.27 1.27)) hide)
     )
@@
       (effects (font (size 1.27 1.27)) (justify right))
     )
-    (property "Value" "" (id 1) (at 114.935 118.11 90)
-      (effects (font (size 1.27 1.27)) (justify right))
-    )
-    (property "Footprint" "" (id 2) (at 123.825 116.205 0)
+    (property "Value" "" (id 1) (at 114.935 117.475 90)
+      (effects (font (size 1.27 1.27)) (justify right))
+    )
+    (property "Footprint" "Connector_PinHeader_2.54mm:PinHeader_1x03_P2.54mm_Horizontal" (id 2) (at 123.825 116.205 0)
       (effects (font (size 1.27 1.27)) hide)
     )
@@
     (in_bom yes) (on_board yes)
     (property "Reference" "TP3" (id 0) (at 88.265 126.365 90))
-    (property "Value" "" (id 1) (at 92.71 126.365 90))
+    (property "Value" "CS" (id 1) (at 92.71 126.365 90))
     (property "Footprint" "TestPoint:TestPoint_Pad_D1.5mm" (id 2) (at 99.06 121.285 0)
       (effects (font (size 1.27 1.27)) hide)
@@
     )
     (path "/90f36d9e-5ac2-402e-9876-8b5aead8f308"
-      (reference "J1") (unit 1) (value "Term") (footprint "Connector_PinHeader_2.54mm:PinHeader_1x03_P2.54mm_Horizontal")
+      (reference "J1") (unit 1) (value "Conn") (footprint "Connector_PinHeader_2.54mm:PinHeader_1x03_P2.54mm_Horizontal")
     )
     (path "/1e76e1cf-4b69-437a-9b31-98a34bc012c8"

Commit message: Work in progress.
Parts:
- J1: value (none) -> Conn
- SW1: footprint Button_Switch_SMD:SW_DIP_SPSTx04_Slide_KingTek_DSHP04TS_W7.62mm_P1.27mm -> Button_Switch_SMD:SW_DIP_SPSTx04_Slide_6.7x11.72mm_W8.61mm_P2.54mm_LowProfile
Connections:
- net A13: now also J1.3 (Pin_3); no longer J1.2 (Pin_2)
- net A14: now also J1.2 (Pin_2); no longer J1.3 (Pin_3)
- net WE: now reaches JP4.2 (B), SW1.4, TP4.1, U1.27 (~{WE})
- net CS: now reaches JP3.2 (B), SW1.3, TP3.1, U1.20 (~{CS})
- net OE: now reaches CN1.20 (/CE), U1.22 (~{OE})
Changed lines of the file:
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@@
   (junction (at 161.29 150.495) (diameter 0) (color 0 0 0 0)
   )
+  (junction (at 126.365 131.445) (diameter 0) (color 0 0 0 0)
+  )
   (junction (at 105.41 126.365) (diameter 0) (color 0 0 0 0)
   )
-  (junction (at 126.365 128.905) (diameter 0) (color 0 0 0 0)
-  )
   (junction (at 139.065 131.445) (diameter 0) (color 0 0 0 0)
   )
   (junction (at 136.525 150.495) (diameter 0) (color 0 0 0 0)
   )
-  (junction (at 123.825 131.445) (diameter 0) (color 0 0 0 0)
-  )
   (junction (at 136.525 128.905) (diameter 0) (color 0 0 0 0)
   )
@@
   (junction (at 136.525 105.41) (diameter 0) (color 0 0 0 0)
   )
+  (junction (at 123.825 128.905) (diameter 0) (color 0 0 0 0)
+  )
   (junction (at 110.49 150.495) (diameter 0) (color 0 0 0 0)
   )
@@
     (stroke (width 0) (type default) (color 0 0 0 0))
   )
-  (wire (pts (xy 126.365 128.905) (xy 136.525 128.905))
+  (wire (pts (xy 110.49 128.905) (xy 123.825 128.905))
     (stroke (width 0) (type default) (color 0 0 0 0))
   )
@@
     (stroke (width 0) (type default) (color 0 0 0 0))
   )
+  (wire (pts (xy 126.365 121.285) (xy 126.365 131.445))
+    (stroke (width 0) (type default) (color 0 0 0 0))
+  )
   (bus (pts (xy 53.34 90.805) (xy 53.34 93.345))
     (stroke (width 0) (type default) (color 0 0 0 0))
@@
     (stroke (width 0) (type default) (color 0 0 0 0))
   )
-  (wire (pts (xy 123.825 121.285) (xy 123.825 131.445))
-    (stroke (width 0) (type default) (color 0 0 0 0))
-  )
   (wire (pts (xy 114.3 113.03) (xy 151.13 113.03))
     (stroke (width 0) (type default) (color 0 0 0 0))
@@
     (stroke (width 0) (type default) (color 0 0 0 0))
   )
-  (wire (pts (xy 110.49 128.905) (xy 126.365 128.905))
-    (stroke (width 0) (type default) (color 0 0 0 0))
-  )
   (wire (pts (xy 148.59 87.63) (xy 151.13 87.63))
     (stroke (width 0) (type default) (color 0 0 0 0))
@@
     (stroke (width 0) (type default) (color 0 0 0 0))
   )
+  (wire (pts (xy 123.825 121.285) (xy 123.825 128.905))
+    (stroke (width 0) (type default) (color 0 0 0 0))
+  )
   (wire (pts (xy 131.445 150.495) (xy 131.445 149.225))
     (stroke (width 0) (type default) (color 0 0 0 0))
   )
+  (wire (pts (xy 126.365 131.445) (xy 139.065 131.445))
+    (stroke (width 0) (type default) (color 0 0 0 0))
+  )
   (wire (pts (xy 55.88 95.885) (xy 57.785 95.885))
     (stroke (width 0) (type default) (color 0 0 0 0))
@@
     (stroke (width 0) (type default) (color 0 0 0 0))
   )
-  (wire (pts (xy 123.825 131.445) (xy 139.065 131.445))
-    (stroke (width 0) (type default) (color 0 0 0 0))
-  )
   (wire (pts (xy 84.455 82.55) (xy 114.3 82.55))
     (stroke (width 0) (type default) (color 0 0 0 0))
@@
     (stroke (width 0) (type default) (color 0 0 0 0))
   )
-  (wire (pts (xy 126.365 121.285) (xy 126.365 128.905))
-    (stroke (width 0) (type default) (color 0 0 0 0))
-  )
   (wire (pts (xy 148.59 77.47) (xy 151.13 77.47))
     (stroke (width 0) (type default) (color 0 0 0 0))
@@
     (stroke (width 0) (type default) (color 0 0 0 0))
   )
+  (wire (pts (xy 123.825 128.905) (xy 136.525 128.905))
+    (stroke (width 0) (type default) (color 0 0 0 0))
+  )
   (bus (pts (xy 146.05 74.93) (xy 146.05 77.47))
     (stroke (width 0) (type default) (color 0 0 0 0))
@@
     (stroke (width 0) (type default) (color 0 0 0 0))
   )
-  (wire (pts (xy 115.57 131.445) (xy 123.825 131.445))
+  (wire (pts (xy 115.57 131.445) (xy 126.365 131.445))
     (stroke (width 0) (type default) (color 0 0 0 0))
   )
@@
     (effects (font (size 1.27 1.27)) (justify right bottom))
   )
+  (label "WE" (at 151.13 110.49 180)
+    (effects (font (size 1.27 1.27)) (justify right bottom))
+  )
   (label "A11" (at 151.13 97.79 180)
     (effects (font (size 1.27 1.27)) (justify right bottom))
@@
     (effects (font (size 1.27 1.27)) (justify right bottom))
   )
+  (label "OE" (at 151.13 113.03 180)
+    (effects (font (size 1.27 1.27)) (justify right bottom))
+  )
   (label "A7" (at 57.785 70.485 180)
     (effects (font (size 1.27 1.27)) (justify right bottom))
@@
   )
   (label "D[0..7]" (at 176.53 164.465 180)
+    (effects (font (size 1.27 1.27)) (justify right bottom))
+  )
+  (label "CS" (at 151.13 115.57 180)
     (effects (font (size 1.27 1.27)) (justify right bottom))
   )
@@
       (effects (font (size 1.27 1.27)) (justify left))
     )
-    (property "Footprint" "Button_Switch_SMD:SW_DIP_SPSTx04_Slide_KingTek_DSHP04TS_W7.62mm_P1.27mm" (id 2) (at 133.985 141.605 0)
+    (property "Footprint" "Button_Switch_SMD:SW_DIP_SPSTx04_Slide_6.7x11.72mm_W8.61mm_P2.54mm_LowProfile" (id 2) (at 133.985 141.605 0)
       (effects (font (size 1.27 1.27)) hide)
     )
@@
       (effects (font (size 1.27 1.27)) (justify right))
     )
-    (property "Value" "" (id 1) (at 114.935 117.475 90)
+    (property "Value" "Conn" (id 1) (at 114.935 117.475 90)
       (effects (font (size 1.27 1.27)) (justify right))
     )
@@
     )
     (path "/6191a81e-6329-4edb-9700-50f6543f797f"
-      (reference "SW1") (unit 1) (value "DIP Switch") (footprint "Button_Switch_SMD:SW_DIP_SPSTx04_Slide_KingTek_DSHP04TS_W7.62mm_P1.27mm")
+      (reference "SW1") (unit 1) (value "DIP Switch") (footprint "Button_Switch_SMD:SW_DIP_SPSTx04_Slide_6.7x11.72mm_W8.61mm_P2.54mm_LowProfile")
     )
     (path "/edce838d-2d8d-4a5f-9a5f-c4ba586d1014"
