File: Compact23256.kicad_pcb (KiCad board)
At the start: 2 copper layers, 18.3 x 31 mm, 15 parts, among them CN1 2364, J1 Term, SW1 DIP Switch, U1 28C256

Commit message: Work in progress.
Parts:
- J1: value Term -> Conn
- moved SW1 0.51 mm to (118.4, 67.8)
Routing:
- net GND: track 0.00 -> 50.3 mm, vias 0 -> 1
- net /A13: track 0.00 -> 46.1 mm, vias 0 -> 5
- net /A14: track 0.00 -> 43.3 mm, vias 0 -> 4
- net Net-(JP3-Pad2): track 0.00 -> 38.8 mm, vias 0 -> 2
- net Net-(JP4-Pad2): track 0.00 -> 26.6 mm, vias 0 -> 3
- net +5V: track 0.00 -> 22.7 mm, vias 0 -> 1
- net /A9: track 0.00 -> 17.5 mm
- net /A6: track 0.00 -> 17.3 mm
- net /D5: track 0.00 -> 17.2 mm
- net /D2: track 0.00 -> 17.2 mm
- net /A7: track 0.00 -> 17.0 mm
- net /A8: track 0.00 -> 16.2 mm, vias 0 -> 1
- net /A11: track 0.00 -> 16.0 mm, vias 0 -> 2
- net /D6: track 0.00 -> 15.9 mm
- net /D1: track 0.00 -> 15.9 mm
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
Commit message: Work in progress.
Parts:
- SW1: footprint Button_Switch_SMD:SW_DIP_SPSTx04_Slide_KingTek_DSHP04TS_W7.62mm_P1.27mm -> Button_Switch_SMD:SW_DIP_SPSTx04_Slide_6.7x11.72mm_W8.61mm_P2.54mm_LowProfile
- moved TP4 10.5 mm to (123.4, 85.3)
- moved JP4 7.27 mm to (122.2, 69.6), turned to -90 degrees
- moved JP1 7.27 mm to (114.6, 69.6), turned to -90 degrees
- moved JP2 3.81 mm to (117.1, 69.6), turned to -90 degrees
- moved JP3 3.81 mm to (119.6, 69.6), turned to -90 degrees
- moved TP1 3.59 mm to (115.8, 85.3)
- moved TP2 3.59 mm to (118.4, 85.3)
- moved TP3 2.54 mm to (120.9, 85.3)
- moved SW1 1.02 mm to (118.4, 68.8), turned to 90 degrees
Connections:
- net Net-(CN1-Pad20) renamed /OE
- net Net-(JP3-Pad2) renamed /CS
- net Net-(JP4-Pad2) renamed /WE
- J1 pad 2: /A13 -> /A14
- J1 pad 3: /A14 -> /A13
Routing:
- net GND: track 50.3 -> 80.5 mm, vias 1 -> 5
- net /CS: track 38.8 -> 22.8 mm
- net /A14: track 43.3 -> 32.1 mm, vias 4 -> 2
- net /A13: track 46.1 -> 36.7 mm, vias 5 -> 4
- net +5V: track 22.7 -> 27.2 mm
- net /D4: track 15.0 -> 18.5 mm, vias 1 -> 0
- net /A11: track 16.0 -> 17.6 mm, vias 2 -> 1
- net /WE: track 26.6 -> 27.9 mm, vias 3 -> 2
- net /D3: track 15.5 -> 16.5 mm, vias 1 -> 0
Other:
- board text added: "A13"
- board text added: "A14"
- board text added: "GND"

Commit message: Work in progress.
Parts:
- moved G*** 17.6 mm to (128.3, 94.7)
- moved J1 2.54 mm to (120.9, 87.9)
Routing:
- net GND: track 80.5 -> 76.5 mm
- net /A14: track 32.1 -> 29.6 mm
- net /A13: track 36.7 -> 34.2 mm
Changed lines of the file:
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@@
   )
   (footprint "Logo:bigby3" (layer "F.Cu")
-    (at 141.224 82.804)
+    (at 128.27 94.742)
     (attr through_hole)
     (fp_text reference "G***" (at 0 0) (layer "F.SilkS") hide
@@
   )
   (footprint "Connector_PinHeader_2.54mm:PinHeader_1x03_P2.54mm_Horizontal" (layer "F.Cu")
-    (at 120.904 90.424 -90)
+    (at 120.904 87.884 -90)
     (descr "Through hole angled pin header, 1x03, 2.54mm pitch, 6mm pin length, single row")
     (tags "Through hole angled pin header THT 1x03 2.54mm single row")
@@
       (effects (font (size 1 1) (thickness 0.15)) (justify mirror))
     )
-    (fp_text value "WE" (at 0 -1.905) (layer "B.SilkS")
+    (fp_text value "WE" (at 0 1.524) (layer "B.Fab")
       (effects (font (size 0.8 0.8) (thickness 0.15)) (justify mirror))
     )
@@
     (property "Sheetname" "")
     (attr smd)
-    (fp_text reference "U1" (at 0 7.62) (layer "B.SilkS")
+    (fp_text reference "U1" (at 0 5.087322) (layer "B.SilkS")
       (effects (font (size 1 1) (thickness 0.15)) (justify mirror))
     )
@@
       (effects (font (size 1 1) (thickness 0.15)) (justify mirror))
     )
-    (fp_text value "A13" (at 0 -1.905) (layer "B.SilkS")
+    (fp_text value "A13" (at 0 1.524) (layer "B.Fab")
       (effects (font (size 0.8 0.8) (thickness 0.15)) (justify mirror))
     )
@@
       (effects (font (size 1 1) (thickness 0.15)) (justify mirror))
     )
-    (fp_text value "CS" (at 0 -1.905) (layer "B.SilkS")
+    (fp_text value "CS" (at 0 1.524) (layer "B.Fab")
       (effects (font (size 0.8 0.8) (thickness 0.15)) (justify mirror))
     )
@@
       (effects (font (size 1 1) (thickness 0.15)) (justify mirror))
     )
-    (fp_text value "A14" (at 0 -1.905) (layer "B.SilkS")
+    (fp_text value "A14" (at 0 1.524) (layer "B.Fab")
       (effects (font (size 0.8 0.8) (thickness 0.15)) (justify mirror))
     )
@@
       (net 24 "/A14") (pinfunction "1") (pintype "passive"))
   )
+  (gr_poly
+    (pts
+      (xy 124.46 83.312)
+      (xy 112.268 83.312)
+      (xy 112.268 76.454)
+      (xy 124.46 76.454)
+    ) (layer "F.SilkS") (width 0.15) (fill solid))
   (gr_line (start 127.508 60.96) (end 127.508 91.948) (layer "Edge.Cuts") (width 0.1))
   (gr_line (start 127.508 91.948) (end 109.22 91.948) (layer "Edge.Cuts") (width 0.1))
   (gr_line (start 109.22 60.96) (end 127.508 60.96) (layer "Edge.Cuts") (width 0.1))
   (gr_line (start 109.22 91.948) (end 109.22 60.96) (layer "Edge.Cuts") (width 0.1))
-  (gr_text "GND" (at 120.904 88.392) (layer "F.SilkS")
+  (gr_text "GND" (at 120.904 86.36) (layer "F.SilkS")
     (effects (font (size 0.8 0.7) (thickness 0.15)))
   )
-  (gr_text "A13" (at 115.824 88.392) (layer "F.SilkS")
+  (gr_text "A13" (at 115.824 86.36) (layer "F.SilkS")
     (effects (font (size 0.8 0.7) (thickness 0.15)))
   )
-  (gr_text "A14" (at 118.364 88.392) (layer "F.SilkS")
+  (gr_text "A14" (at 118.364 86.36) (layer "F.SilkS")
     (effects (font (size 0.8 0.7) (thickness 0.15)))
   )
@@
   (segment (start 119.634 64.529) (end 120.355489 65.250489) (width 0.35) (layer "F.Cu") (net 12))
   (segment (start 123.698 75.067436) (end 123.698 64.008) (width 0.35) (layer "F.Cu") (net 12))
-  (segment (start 120.904 90.424) (end 122.047 89.281) (width 0.35) (layer "F.Cu") (net 12))
-  (segment (start 122.047 89.281) (end 122.047 88.773) (width 0.35) (layer "F.Cu") (net 12))
   (segment (start 118.11 65.545) (end 117.094 64.529) (width 0.35) (layer "F.Cu") (net 12))
+  (segment (start 120.904 87.884) (end 122.174 87.884) (width 0.35) (layer "F.Cu") (net 12))
   (segment (start 120.355489 65.250489) (end 120.355489 66.347943) (width 0.35) (layer "F.Cu") (net 12))
   (segment (start 114.554 68.946) (end 114.554 64.529) (width 0.35) (layer "F.Cu") (net 12))
   (segment (start 115.57 65.545) (end 114.554 64.529) (width 0.35) (layer "F.Cu") (net 12))
+  (segment (start 123.444 87.884) (end 124.714 86.614) (width 0.35) (layer "F.Cu") (net 12))
   (segment (start 124.714 86.614) (end 124.714 76.083436) (width 0.35) (layer "F.Cu") (net 12))
-  (segment (start 122.047 88.773) (end 122.047 83.693) (width 0.35) (layer "F.Cu") (net 12))
   (segment (start 115.57 66.421) (end 115.57 65.545) (width 0.35) (layer "F.Cu") (net 12))
   (segment (start 124.714 76.083436) (end 123.698 75.067436) (width 0.35) (layer "F.Cu") (net 12))
+  (segment (start 122.174 83.566) (end 122.174 87.884) (width 0.35) (layer "F.Cu") (net 12))
   (segment (start 119.634 68.946) (end 119.634 64.529) (width 0.35) (layer "F.Cu") (net 12))
-  (segment (start 120.904 90.424) (end 124.714 86.614) (width 0.35) (layer "F.Cu") (net 12))
   (segment (start 117.094 68.946) (end 117.094 64.529) (width 0.35) (layer "F.Cu") (net 12))
-  (segment (start 122.047 83.693) (end 122.174 83.566) (width 0.35) (layer "F.Cu") (net 12))
-  (via (at 122.174 83.566) (size 0.8) (drill 0.4) (layers "F.Cu" "B.Cu") (net 12))
+  (segment (start 122.174 87.884) (end 123.444 87.884) (width 0.35) (layer "F.Cu") (net 12))
   (via (at 115.57 66.421) (size 0.8) (drill 0.4) (layers "F.Cu" "B.Cu") (net 12))
   (via (at 120.355489 66.347943) (size 0.8) (drill 0.4) (layers "F.Cu" "B.Cu") (net 12))
+  (via (at 122.174 83.566) (size 0.8) (drill 0.4) (layers "F.Cu" "B.Cu") (net 12))
   (via (at 118.11 66.421) (size 0.8) (drill 0.4) (layers "F.Cu" "B.Cu") (net 12))
   (via (at 123.698 64.008) (size 0.8) (drill 0.4) (layers "F.Cu" "B.Cu") (net 12))
@@
   (segment (start 122.174 83.566) (end 122.174 83.517) (width 0.35) (layer "B.Cu") (net 12))
   (segment (start 118.11 66.421) (end 120.282432 66.421) (width 0.35) (layer "B.Cu") (net 12))
+  (segment (start 118.364 90.424) (end 120.904 87.884) (width 0.35) (layer "B.Cu") (net 12))
+  (segment (start 110.744 90.424) (end 118.364 90.424) (width 0.35) (layer "B.Cu") (net 12))
   (segment (start 123.698 64.008) (end 122.11548 62.42548) (width 0.35) (layer "B.Cu") (net 12))
   (segment (start 120.282432 66.421) (end 120.355489 66.347943) (width 0.35) (layer "B.Cu") (net 12))
-  (segment (start 110.744 90.424) (end 111.968511 91.648511) (width 0.35) (layer "B.Cu") (net 12))
-  (segment (start 111.968511 91.648511) (end 119.679489 91.648511) (width 0.35) (layer "B.Cu") (net 12))
   (segment (start 122.174 83.517) (end 123.014 82.677) (width 0.35) (layer "B.Cu") (net 12))
   (segment (start 120.65 66.053432) (end 120.355489 66.347943) (width 0.35) (layer "B.Cu") (net 12))
   (segment (start 122.11548 62.42548) (end 121.041316 62.42548) (width 0.35) (layer "B.Cu") (net 12))
-  (segment (start 119.679489 91.648511) (end 120.904 90.424) (width 0.35) (layer "B.Cu") (net 12))
-  (segment (start 124.556335 90.424) (end 125.984 90.424) (width 0.2) (layer "B.Cu") (net 13))
   (segment (start 118.491 82.677) (end 119.894489 84.080489) (width 0.2) (layer "B.Cu") (net 13))
+  (segment (start 119.894489 85.762154) (end 120.866824 86.734489) (width 0.2) (layer "B.Cu") (net 13))
   (segment (start 113.714 82.677) (end 118.491 82.677) (width 0.2) (layer "B.Cu") (net 13))
-  (segment (start 119.894489 85.762154) (end 124.556335 90.424) (width 0.2) (layer "B.Cu") (net 13))
+  (segment (start 122.294489 86.734489) (end 125.984 90.424) (width 0.2) (layer "B.Cu") (net 13))
+  (segment (start 120.866824 86.734489) (end 122.294489 86.734489) (width 0.2) (layer "B.Cu") (net 13))
   (segment (start 119.894489 84.080489) (end 119.894489 85.762154) (width 0.2) (layer "B.Cu") (net 13))
   (segment (start 124.46 82.462283) (end 124.46 84.423909) (width 0.2) (layer "B.Cu") (net 14))
@@
   (segment (start 121.539 67.307852) (end 121.539 67.31) (width 0.2) (layer "B.Cu") (net 24))
   (segment (start 120.904 67.945) (end 118.491 67.945) (width 0.2) (layer "B.Cu") (net 24))
+  (segment (start 118.364 87.884) (end 118.364 85.344) (width 0.2) (layer "B.Cu") (net 24))
   (segment (start 123.014 64.9515) (end 121.5625 63.5) (width 0.2) (layer "B.Cu") (net 24))
   (segment (start 123.014 66.167) (end 122.679852 66.167) (width 0.2) (layer "B.Cu") (net 24))
   (segment (start 121.539 67.31) (end 120.904 67.945) (width 0.2) (layer "B.Cu") (net 24))
-  (segment (start 118.364 85.344) (end 118.364 90.424) (width 0.2) (layer "B.Cu") (net 24))
   (segment (start 122.679852 66.167) (end 121.539 67.307852) (width 0.2) (layer "B.Cu") (net 24))
   (segment (start 118.364 85.344) (end 118.364 84.074) (width 0.2) (layer "B.Cu") (net 24))
@@
   (segment (start 116.9905 62.8885) (end 116.9905 63.5) (width 0.2) (layer "B.Cu") (net 25))
   (segment (start 113.714 68.707) (end 112.286488 68.707) (width 0.2) (layer "B.Cu") (net 25))
-  (segment (start 115.824 85.344) (end 115.824 90.424) (width 0.2) (layer "B.Cu") (net 25))
   (segment (start 116.586 62.484) (end 116.9905 62.8885) (width 0.2) (layer "B.Cu") (net 25))
   (segment (start 113.714 68.707) (end 115.189 68.707) (width 0.2) (layer "B.Cu") (net 25))
   (segment (start 115.824 85.344) (end 115.824 84.074) (width 0.2) (layer "B.Cu") (net 25))
+  (segment (start 115.824 87.884) (end 115.824 85.344) (width 0.2) (layer "B.Cu") (net 25))
   (segment (start 112.286488 68.707) (end 112.213744 68.634256) (width 0.2) (layer "B.Cu") (net 25))
   (segment (start 114.958636 73.638086) (end 115.169234 73.427489) (width 0.2) (layer "B.Cu") (net 26))

Commit message: Work in progress.
Parts:
- removed the G*** at (128.3, 94.7)
- added G***: LOGO, Logo:bigby3-cu, F.Cu at (113.3, 84.8)
Other:
- board text added: "KERNALquattro"
Changed lines of the file:
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@@
       (net 28 "/WE") (pinfunction "B") (pintype "passive"))
   )
-  (footprint "Logo:bigby3" (layer "F.Cu")
-    (at 128.27 94.742)
+  (footprint "Library:SolderJumper-2_slim" (layer "F.Cu")
+    (at 119.634 69.596 -90)
+    (descr "SMD Solder Jumper, half width, open")
+    (tags "solder jumper open")
+    (property "Sheetfile" "Compact23256.kicad_sch")
+    (property "Sheetname" "")
+    (attr exclude_from_pos_files)
+    (fp_text reference "JP3" (at 0 -1.3 90) (layer "F.SilkS") hide
+      (effects (font (size 1 1) (thickness 0.15)))
+    )
+    (fp_text value "CS" (at -2.159 0 90) (layer "F.SilkS")
+      (effects (font (size 0.8 0.7) (thickness 0.12)))
+    )
+    (fp_line (start -1.3 0.5) (end -0.9 0.5) (layer "F.SilkS") (width 0.1))
+    (fp_line (start 1.3 -0.5) (end 1.3 0.5) (layer "F.SilkS") (width 0.1))
+    (fp_line (start -1.3 0.5) (end -1.3 -0.5) (layer "F.SilkS") (width 0.1))
+    (fp_line (start 0.9 -0.5) (end 1.3 -0.5) (layer "F.SilkS") (width 0.1))
+    (fp_line (start -1.3 -0.5) (end -0.9 -0.5) (layer "F.SilkS") (width 0.1))
+    (fp_line (start 0.9 0.5) (end 1.3 0.5) (layer "F.SilkS") (width 0.1))
+    (fp_line (start 1.4 0.6) (end 1.4 -0.6) (layer "F.CrtYd") (width 0.05))
+    (fp_line (start -1.4 -0.6) (end 1.4 -0.6) (layer "F.CrtYd") (width 0.05))
+    (fp_line (start -1.4 -0.6) (end -1.4 0.6) (layer "F.CrtYd") (width 0.05))
+    (fp_line (start -1.4 0.6) (end 1.4 0.6) (layer "F.CrtYd") (width 0.05))
+    (pad "1" smd rect (at -0.65 0 270) (size 1 0.75) (layers "F.Cu" "F.Mask")
+      (net 12 "GND") (pinfunction "A") (pintype "passive"))
+    (pad "2" smd rect (at 0.65 0 270) (size 1 0.75) (layers "F.Cu" "F.Mask")
+      (net 27 "/CS") (pinfunction "B") (pintype "passive"))
+  )
+  (footprint "Logo:bigby3-cu" (layer "F.Cu")
+    (at 113.284 84.836)
     (attr through_hole)
     (fp_text reference "G***" (at 0 0) (layer "F.SilkS") hide
@@
         (xy -0.126406 -1.1161)
         (xy -0.026724 -1.11327)
-      ) (layer "F.SilkS") (width 0.01) (fill solid))
-  )
-  (footprint "Library:SolderJumper-2_slim" (layer "F.Cu")
-    (at 119.634 69.596 -90)
-    (descr "SMD Solder Jumper, half width, open")
-    (tags "solder jumper open")
-    (property "Sheetfile" "Compact23256.kicad_sch")
-    (property "Sheetname" "")
-    (attr exclude_from_pos_files)
-    (fp_text reference "JP3" (at 0 -1.3 90) (layer "F.SilkS") hide
-      (effects (font (size 1 1) (thickness 0.15)))
-    )
-    (fp_text value "CS" (at -2.159 0 90) (layer "F.SilkS")
-      (effects (font (size 0.8 0.7) (thickness 0.12)))
-    )
-    (fp_line (start -1.3 0.5) (end -0.9 0.5) (layer "F.SilkS") (width 0.1))
-    (fp_line (start 1.3 -0.5) (end 1.3 0.5) (layer "F.SilkS") (width 0.1))
-    (fp_line (start -1.3 0.5) (end -1.3 -0.5) (layer "F.SilkS") (width 0.1))
-    (fp_line (start 0.9 -0.5) (end 1.3 -0.5) (layer "F.SilkS") (width 0.1))
-    (fp_line (start -1.3 -0.5) (end -0.9 -0.5) (layer "F.SilkS") (width 0.1))
-    (fp_line (start 0.9 0.5) (end 1.3 0.5) (layer "F.SilkS") (width 0.1))
-    (fp_line (start 1.4 0.6) (end 1.4 -0.6) (layer "F.CrtYd") (width 0.05))
-    (fp_line (start -1.4 -0.6) (end 1.4 -0.6) (layer "F.CrtYd") (width 0.05))
-    (fp_line (start -1.4 -0.6) (end -1.4 0.6) (layer "F.CrtYd") (width 0.05))
-    (fp_line (start -1.4 0.6) (end 1.4 0.6) (layer "F.CrtYd") (width 0.05))
-    (pad "1" smd rect (at -0.65 0 270) (size 1 0.75) (layers "F.Cu" "F.Mask")
-      (net 12 "GND") (pinfunction "A") (pintype "passive"))
-    (pad "2" smd rect (at 0.65 0 270) (size 1 0.75) (layers "F.Cu" "F.Mask")
-      (net 27 "/CS") (pinfunction "B") (pintype "passive"))
+      ) (layer "F.Cu") (width 0.01) (fill solid))
   )
   (footprint "Library:SolderJumper-2_slim" (layer "F.Cu")
@@
     (property "Sheetname" "")
     (attr through_hole)
-    (fp_text reference "CN1" (at 7.62 -2.33) (layer "F.SilkS")
+    (fp_text reference "CN1" (at 7.62 -2.33) (layer "F.SilkS") hide
       (effects (font (size 1 1) (thickness 0.15)))
     )
@@
   (gr_poly
     (pts
-      (xy 124.46 83.312)
-      (xy 112.268 83.312)
-      (xy 112.268 76.454)
-      (xy 124.46 76.454)
+      (xy 124.206 83.312)
+      (xy 112.522 83.312)
+      (xy 112.522 76.454)
+      (xy 124.206 76.454)
     ) (layer "F.SilkS") (width 0.15) (fill solid))
   (gr_line (start 127.508 60.96) (end 127.508 91.948) (layer "Edge.Cuts") (width 0.1))
@@
   (gr_line (start 109.22 60.96) (end 127.508 60.96) (layer "Edge.Cuts") (width 0.1))
   (gr_line (start 109.22 91.948) (end 109.22 60.96) (layer "Edge.Cuts") (width 0.1))
+  (gr_text "KERNALquattro" (at 118.364 90.424) (layer "F.Cu")
+    (effects (font (size 1.1 1.1) (thickness 0.25)))
+  )
   (gr_text "GND" (at 120.904 86.36) (layer "F.SilkS")
     (effects (font (size 0.8 0.7) (thickness 0.15)))
@@
     (effects (font (size 0.8 0.7) (thickness 0.15)))
   )
+  (gr_text "KERNALquattro" (at 118.364 90.424) (layer "F.Mask")
+    (effects (font (size 1.1 1.1) (thickness 0.25)))
+  )
   (segment (start 112.744852 68.072) (end 112.163022 67.49017) (width 0.2) (layer "B.Cu") (net 1))
