File: KernalQuattro.kicad_sch (KiCad schematic)
At the start: 14 parts, among them CN1 2364, J1 Conn, SW1 DIP Switch, U1 28C256

Commit message: Rounded corners.
Other:
- title: (none) -> KERNALquattro
Changed lines of the file:
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@@
   (paper "A4")
   (title_block
+    (title "KERNALquattro")
     (rev "1")
     (company "www.hackup.net")
