File: KQAdapter/KQAdapter.kicad_pcb (KiCad board)
At the start: 2 copper layers, 20.8 x 36.6 mm, 4 parts, among them CN1 2364, J1 Pogo, U1 28C256

Commit message: Work in progress.
Parts:
- added G***: LOGO, Library:quattro, F.Cu at (108.1, 108.3)
Other:
- outline, holes or cut-outs redrawn
- board text added: "ADAPTER"
- board text added: "KERNAL"
- board text added: "KERNALquattro 28C256 Programming Adapter Rev.1 github.com/hackup/KERNALquattro"
- board text removed: "KERNAL quattro"
